Commit message: Update environment node

File: src/fun4/robot/visual/my-robot.xacro (robot description, xacro)
@@ -1,8 +1,8 @@
 <?xml version="1.0"?>
-<robot xmlns:xacro="http://www.ros.org/wiki/xacro" name="example">
+<robot xmlns:xacro="http://www.ros.org/wiki/xacro" name="RRR">
   <link name="link_0">
     <visual>
       <geometry>
-        <mesh filename="file:///$(find example_description)/meshes/link_0.stl"/>
+        <mesh filename="file:///$(find fun4)/meshes/link_0.stl"/>
       </geometry>
     </visual>
@@ -11,5 +11,5 @@
     <visual>
       <geometry>
-        <mesh filename="file:///$(find example_description)/meshes/link_1.stl"/>
+        <mesh filename="file:///$(find fun4)/meshes/link_1.stl"/>
       </geometry>
     </visual>
@@ -28,7 +28,7 @@
   <link name="link_2">
     <visual>
-      <origin xyz="0.0 0.0 0.0" rpy="0 0 ${-3.14/2}"/>
+      <origin xyz="0.0 0.0 0.0" rpy="3.14 0 0"/>
       <geometry>
-        <mesh filename="file:///$(find example_description)/meshes/link_2.stl"/>
+        <mesh filename="file:///$(find fun4)/meshes/link_2.stl"/>
       </geometry>
     </visual>
@@ -37,5 +37,5 @@
     <parent link="link_1"/>
     <child link="link_2"/>
-    <origin xyz="0.0 -0.12 0.0" rpy="${-3.14/2} 0 0"/>
+    <origin xyz="0.0 -0.12 0.0" rpy="${3.14/2} ${-3.14/2} 0"/>
     <axis xyz="0 0 1"/>
     <limit
@@ -47,7 +47,7 @@
   <link name="link_3">
     <visual>
-      <origin xyz="0.0 0.0 0.0" rpy="0 0 ${-3.14/2}"/>
+      <origin xyz="0.0 0.0 0.0" rpy="3.14 0 ${3.14/2}"/>
       <geometry>
-        <mesh filename="file:///$(find example_description)/meshes/link_3.stl"/>
+        <mesh filename="file:///$(find fun4)/meshes/link_3.stl"/>
       </geometry>
     </visual>
@@ -56,5 +56,5 @@
     <parent link="link_2"/>
     <child link="link_3"/>
-    <origin xyz="0.0 -0.25 0.1" rpy="0 0 0"/>
+    <origin xyz="0.25 0.0 -0.1" rpy="0 0 ${-3.14/2}"/>
     <axis xyz="0 0 1"/>
     <limit
@@ -68,5 +68,5 @@
       <origin xyz="0.0 0.0 0.0" rpy="0 0 0"/>
       <geometry>
-        <mesh filename="file:///$(find example_description)/meshes/end_effector.stl"/>
+        <mesh filename="file:///$(find fun4)/meshes/end_effector.stl"/>
       </geometry>
     </visual>
@@ -75,5 +75,5 @@
     <parent link="link_3"/>
     <child link="end_effector"/>
-    <origin xyz="0.0 -0.28 0.0" rpy="${3.14/2} 0 0"/>
+    <origin xyz="0.0 0.28 0.0" rpy="${-3.14/2} 0 0"/>
   </joint>
 </robot>
